Commit message: ye

File: onshape/urdf_output/robot.urdf (robot description, URDF)
Before this commit: robot robot, 2 links, 1 joints
Joints:
- joint revolute_1: child part_2_1 -> part_1_1; origin xyz=-0.045115367 -0.055396627 0.053246148 rpy=1.5707963 -0.036563565 -3.1415927 -> xyz=-0.04976857 -0.083174522 0.07368213 rpy=-1.5707963 0 0; parent part_1_1 -> part_2_1

Commit message: fixed COM and hardcoded revolute limits

File: onshape/urdf_output/robot.urdf (robot description, URDF)
Before this commit: robot robot, 2 links, 1 joints
Links:
- link part_1_1: mass 1.0 -> 0.56836923
- link part_2_1: mass 1.0 -> 0.57017369
Joints:
- joint revolute_1: child part_1_1 -> part_2_1; limit lower=-3.14159 upper=3.14159 effort=100 velocity=3.14159 -> (none); origin xyz=-0.04976857 -0.083174522 0.07368213 rpy=-1.5707963 0 0 -> xyz=-0.10943506 -0.0096106609 0.10878255 rpy=-1.5707963 1.5707963 0; parent part_2_1 -> part_1_1; type revolute -> continuous

Commit message: can now detect revolute limits, and clears urdf output each run

File: onshape/urdf_output/robot.urdf (robot description, URDF)
Before this commit: robot robot, 2 links, 1 joints
Links:
- added link part_3_1, mass 0.56836923; collision mesh filename=meshes/part_3_1.stl; visual mesh filename=meshes/part_3_1.stl
- link part_2_1: mass 0.57017369 -> 0.56836923
Joints:
- added joint revolute_2: type revolute, parent part_3_1, child part_2_1, origin xyz=0.054246123 0.0043365703 0.12514557 rpy=1.5707963 0 1.5707963, axis 0 0 1, limit lower=4.1887902047863905 upper=6.283185307179586 effort=100 velocity=3.14159
- joint revolute_1: child part_2_1 -> part_1_1; limit (none) -> lower=4.1887902047863905 upper=6.283185307179586 effort=100 velocity=3.14159; origin xyz=-0.10943506 -0.0096106609 0.10878255 rpy=-1.5707963 1.5707963 0 -> xyz=-0.050753877 0.0043365703 0.12514557 rpy=1.5707963 0 1.5707963; parent part_1_1 -> part_3_1; type continuous -> revolute

Commit message: way better initialisation, debugging, note fixed connection makes part names combine in genesis

File: onshape/urdf_output/robot.urdf (robot description, URDF)
Before this commit: robot robot, 3 links, 2 joints
Links:
- added link part_4_1, mass 0.56836923; collision mesh filename=meshes/part_4_1.stl; visual mesh filename=meshes/part_4_1.stl
- added link part_5_1, mass 0.56836923; collision mesh filename=meshes/part_5_1.stl; visual mesh filename=meshes/part_5_1.stl
- added link part_6_1, mass 0.56836923; collision mesh filename=meshes/part_6_1.stl; visual mesh filename=meshes/part_6_1.stl
- added link part_7_1, mass 0.56836923; collision mesh filename=meshes/part_7_1.stl; visual mesh filename=meshes/part_7_1.stl
- added link part_8_1, mass 0.56836923; collision mesh filename=meshes/part_8_1.stl; visual mesh filename=meshes/part_8_1.stl
- added link part_9_1, mass 0.4167289; collision mesh filename=meshes/part_9_1.stl; visual mesh filename=meshes/part_9_1.stl
Joints:
- added joint fastened_1: type fixed, parent part_3_1, child part_4_1, origin xyz=-0.050753877 0.01680688 0.15279361 rpy=3.1415927 0 0
- added joint fastened_2: type fixed, parent part_3_1, child part_5_1, origin xyz=0.054246123 0.01680688 0.15279361 rpy=3.1415927 0 0
- added joint fastened_3: type fixed, parent part_4_1, child part_6_1, origin xyz=0 0 -0.105 rpy=0 0 0
- added joint revolute_3: type continuous, parent part_4_1, child part_7_1, origin xyz=-0.01382402 0 -0.105 rpy=-1.5707963 0 -1.5707963, axis 0 0 1
- added joint revolute_4: type continuous, parent part_5_1, child part_8_1, origin xyz=0.01382402 0 -0.105 rpy=1.5707963 0 -1.5707963, axis 0 0 1
- added joint revolute_5: type revolute, parent part_6_1, child part_9_1, origin xyz=0.0525 0 -0.02764804 rpy=0 0 0, axis 0 0 1, limit lower=0.0017453292519943296 upper=0.0017453292519943296 effort=100 velocity=3.14159

Commit message: seperate robot and car, car ppo tuning

File: onshape/urdf_output/robot.urdf (robot description, URDF)
Before this commit: robot robot, 9 links, 8 joints
Links:
- removed link part_6_1
- removed link part_7_1
- removed link part_8_1
- removed link part_9_1
- link part_1_1: mass 0.56836923 -> 0.1042
- link part_2_1: mass 0.56836923 -> 0.019490441
- link part_3_1: mass 0.56836923 -> 0.019490441
- link part_4_1: mass 0.56836923 -> 0.019490441
- link part_5_1: mass 0.56836923 -> 0.019490441
Joints:
- removed joint fastened_1
- removed joint fastened_2
- removed joint fastened_3
- removed joint revolute_5
- joint revolute_1: child part_1_1 -> part_3_1; limit lower=4.1887902047863905 upper=6.283185307179586 effort=100 velocity=3.14159 -> (none); origin xyz=-0.050753877 0.0043365703 0.12514557 rpy=1.5707963 0 1.5707963 -> xyz=-0.025 -0.0521 0 rpy=1.5707963 0 1.5707963; parent part_3_1 -> part_1_1; type revolute -> continuous
- joint revolute_2: limit lower=4.1887902047863905 upper=6.283185307179586 effort=100 velocity=3.14159 -> (none); origin xyz=0.054246123 0.0043365703 0.12514557 rpy=1.5707963 0 1.5707963 -> xyz=0.025 -0.0521 0 rpy=-1.5707963 0 1.5707963; parent part_3_1 -> part_1_1; type revolute -> continuous
- joint revolute_3: child part_7_1 -> part_4_1; origin xyz=-0.01382402 0 -0.105 rpy=-1.5707963 0 -1.5707963 -> xyz=0.025 0.0521 0 rpy=-1.5707963 0 1.5707963; parent part_4_1 -> part_1_1
- joint revolute_4: child part_8_1 -> part_5_1; origin xyz=0.01382402 0 -0.105 rpy=1.5707963 0 -1.5707963 -> xyz=-0.025 0.0521 0 rpy=1.5707963 0 1.5707963; parent part_5_1 -> part_1_1
